Commit message: add human occupancy

File: src/ur_description/urdf/simplehumanurdf.urdf (robot description, URDF)
Before this commit: robot test_robot, 7 links, 6 joints
Links:
- removed link base_corps_link_1
- removed link base_corps_link_2
- removed link left_arm_shoulder
- removed link left_forearm
- removed link left_shoulder_psi_link
- removed link link_virtual
- removed link world
- added link base_link; visual box size=0.15 0.1 0.8
- added link right_upper_arm_virtual_1; visual box size=0.001 0.001 0.001
Joints:
- removed joint joint1
- removed joint joint2
- removed joint joint3
- removed joint joint_chest_y
- removed joint joint_chest_z
- removed joint world_joint
- added joint base_to_virtual1: type continuous, parent base_link, child right_upper_arm_virtual_1, origin xyz=-0.05 -0.0725 0.4, axis 0 -1 0
